File: kiosk/electronics/iowa-rover-kiosk-lamps/iowa-rover-kiosk-lamps.kicad_pcb (KiCad board)
At the start: 2 copper layers, 87.6 x 36.8 mm, 16 parts, among them J1 Conn_01x08, SW1 SW_Push, U1 TPIC6B595

Commit message: update
Parts:
- Error Lamp: renamed from LA6
- RFID Lamp 1: renamed from LA1
- RFID Lamp 2: renamed from LA2
- RFID Lamp 3: renamed from LA3
- RFID Lamp 4: renamed from LA4
- Ready Lamp: renamed from LA5
- Running Lamp: renamed from LA7
- Tx Btn: renamed from SW1
- Tx Btn Lamp: renamed from LA8
Connections:
- Tx Btn Lamp pad 1: +12V -> +5V
Routing:
- net +5V: track 76.3 -> 98.1 mm
- net +12V: track 129.4 -> 126.8 mm
- net Net-(J1-Pin_6): track 25.3 -> 26.2 mm
Other:
- board text added: "+"
Changed lines of the file:
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@@
     (property "ki_keywords" "lamp")
     (attr through_hole)
-    (fp_text reference "LA2" (at 2.54 -5.08) (layer "F.SilkS")
+    (fp_text reference "RFID Lamp 2" (at 2.54 -5.08) (layer "F.SilkS")
         (effects (font (size 1 1) (thickness 0.15)))
     )
@@
     (property "ki_keywords" "lamp")
     (attr through_hole)
-    (fp_text reference "LA4" (at 2.54 -5.08) (layer "F.SilkS")
+    (fp_text reference "RFID Lamp 4" (at 2.54 -5.08) (layer "F.SilkS")
         (effects (font (size 1 1) (thickness 0.15)))
     )
@@
     (property "ki_keywords" "lamp")
     (attr through_hole)
-    (fp_text reference "LA6" (at 2.54 -5.08) (layer "F.SilkS")
+    (fp_text reference "Error Lamp" (at 2.54 -5.08) (layer "F.SilkS")
         (effects (font (size 1 1) (thickness 0.15)))
     )
@@
     (property "ki_keywords" "switch normally-open pushbutton push-button")
     (attr through_hole)
-    (fp_text reference "SW1" (at 1.905 -5.08) (layer "F.SilkS")
+    (fp_text reference "Tx Btn" (at 1.905 -5.08) (layer "F.SilkS")
         (effects (font (size 1 1) (thickness 0.15)))
     )
@@
     (property "ki_keywords" "lamp")
     (attr through_hole)
-    (fp_text reference "LA8" (at 2.54 -5.08) (layer "F.SilkS")
+    (fp_text reference "Tx Btn Lamp" (at 2.54 -5.08) (layer "F.SilkS")
         (effects (font (size 1 1) (thickness 0.15)))
     )
@@
       (stroke (width 0.1) (type solid)) (layer "F.Fab"))
     (pad "1" thru_hole rect (at 0 0 180) (size 3 3) (drill 1.52) (layers "*.Cu" "*.Mask")
-      (net 2 "+12V") (pinfunction "-") (pintype "passive"))
+      (net 3 "+5V") (pinfunction "-") (pintype "passive"))
     (pad "2" thru_hole circle (at 5.08 0 180) (size 3 3) (drill 1.52) (layers "*.Cu" "*.Mask")
       (net 19 "Net-(LA8-+)") (pinfunction "+") (pintype "passive"))
@@
     (property "ki_keywords" "lamp")
     (attr through_hole)
-    (fp_text reference "LA5" (at 1.905 -5.08) (layer "F.SilkS")
+    (fp_text reference "Ready Lamp" (at 1.905 -5.08) (layer "F.SilkS")
         (effects (font (size 1 1) (thickness 0.15)))
     )
@@
     (property "ki_keywords" "lamp")
     (attr through_hole)
-    (fp_text reference "LA7" (at 1.905 -5.08) (layer "F.SilkS")
+    (fp_text reference "Running Lamp" (at 1.905 -5.08) (layer "F.SilkS")
         (effects (font (size 1 1) (thickness 0.15)))
     )
@@
     (property "ki_keywords" "lamp")
     (attr through_hole)
-    (fp_text reference "LA1" (at 1.905 -5.08) (layer "F.SilkS")
+    (fp_text reference "RFID Lamp 1" (at 1.905 -5.08) (layer "F.SilkS")
         (effects (font (size 1 1) (thickness 0.15)))
     )
@@
     (property "ki_keywords" "lamp")
     (attr through_hole)
-    (fp_text reference "LA3" (at 1.905 -5.08) (layer "F.SilkS")
+    (fp_text reference "RFID Lamp 3" (at 1.905 -5.08) (layer "F.SilkS")
         (effects (font (size 1 1) (thickness 0.15)))
     )
@@
   (gr_line (start 74.295 33.02) (end 74.295 63.5)
     (stroke (width 0.1) (type default)) (layer "Edge.Cuts"))
+  (gr_text "+\n" (at 101.092 44.196) (layer "F.SilkS")
+    (effects (font (size 1.5 1.5) (thickness 0.3) bold) (justify left bottom mirror))
+  )
+  (gr_text "+\n" (at 156.972 32.004) (layer "F.SilkS")
+    (effects (font (size 1.5 1.5) (thickness 0.3) bold) (justify left bottom mirror))
+  )
+  (gr_text "+\n" (at 93.726 32.004) (layer "F.SilkS")
+    (effects (font (size 1.5 1.5) (thickness 0.3) bold) (justify left bottom mirror))
+  )
+  (gr_text "+\n" (at 148.844 44.196) (layer "F.SilkS")
+    (effects (font (size 1.5 1.5) (thickness 0.3) bold) (justify left bottom mirror))
+  )
+  (gr_text "+\n" (at 132.842 44.196) (layer "F.SilkS")
+    (effects (font (size 1.5 1.5) (thickness 0.3) bold) (justify left bottom mirror))
+  )
+  (gr_text "+\n" (at 125.476 32.004) (layer "F.SilkS")
+    (effects (font (size 1.5 1.5) (thickness 0.3) bold) (justify left bottom mirror))
+  )
+  (gr_text "+\n" (at 109.474 32.004) (layer "F.SilkS")
+    (effects (font (size 1.5 1.5) (thickness 0.3) bold) (justify left bottom mirror))
+  )
+  (gr_text "+\n" (at 117.094 44.196) (layer "F.SilkS")
+    (effects (font (size 1.5 1.5) (thickness 0.3) bold) (justify left bottom mirror))
+  )
+  (gr_text "+\n" (at 141.224 32.004) (layer "F.SilkS")
+    (effects (font (size 1.5 1.5) (thickness 0.3) bold) (justify left bottom mirror))
+  )
   (segment (start 120.65 34.29) (end 122.6 32.34) (width 0.5) (layer "F.Cu") (net 2))
   (segment (start 134.575 32.34) (end 136.525 34.29) (width 0.5) (layer "F.Cu") (net 2))
@@
   (segment (start 102.825 32.34) (end 104.775 34.29) (width 0.5) (layer "F.Cu") (net 2))
   (segment (start 88.9 34.29) (end 90.85 32.34) (width 0.5) (layer "F.Cu") (net 2))
-  (segment (start 144.145 41.91) (end 144.145 46.355) (width 0.5) (layer "F.Cu") (net 2))
   (segment (start 118.7 32.34) (end 120.65 34.29) (width 0.5) (layer "F.Cu") (net 2))
   (segment (start 104.775 34.29) (end 112.395 41.91) (width 0.5) (layer "F.Cu") (net 2))
   (segment (start 112.395 41.91) (end 112.395 46.355) (width 0.5) (layer "F.Cu") (net 2))
   (segment (start 104.775 34.29) (end 106.725 32.34) (width 0.5) (layer "F.Cu") (net 2))
-  (segment (start 136.525 34.29) (end 144.145 41.91) (width 0.5) (layer "F.Cu") (net 2))
   (segment (start 90.85 32.34) (end 102.825 32.34) (width 0.5) (layer "F.Cu") (net 2))
   (segment (start 88.9 34.29) (end 96.52 41.91) (width 0.5) (layer "F.Cu") (net 2))
   (segment (start 122.6 32.34) (end 134.575 32.34) (width 0.5) (layer "F.Cu") (net 2))
-  (segment (start 134.63 55.87) (end 144.145 46.355) (width 0.5) (layer "B.Cu") (net 2))
-  (segment (start 134.63 58.425) (end 134.63 55.87) (width 0.5) (layer "B.Cu") (net 2))
+  (segment (start 134.63 58.425) (end 141.015 52.04) (width 0.5) (layer "B.Cu") (net 2))
+  (segment (start 141.015 38.78) (end 136.525 34.29) (width 0.5) (layer "B.Cu") (net 2))
+  (segment (start 141.015 52.04) (end 141.015 38.78) (width 0.5) (layer "B.Cu") (net 2))
   (segment (start 131.83 66.305) (end 103.135 66.305) (width 0.25) (layer "F.Cu") (net 3))
-  (segment (start 152.4 52.56637) (end 142.82637 62.14) (width 0.25) (layer "F.Cu") (net 3))
+  (segment (start 140.196701 62.14) (end 140.97 61.366701) (width 0.25) (layer "F.Cu") (net 3))
+  (segment (start 138.345 62.14) (end 140.196701 62.14) (width 0.25) (layer "F.Cu") (net 3))
+  (segment (start 147.156 62.14) (end 152.4 56.896) (width 0.25) (layer "F.Cu") (net 3))
   (segment (start 137.17 60.965) (end 131.83 66.305) (width 0.25) (layer "F.Cu") (net 3))
-  (segment (start 138.345 62.14) (end 137.17 60.965) (width 0.25) (layer "F.Cu") (net 3))
-  (segment (start 142.82637 62.14) (end 138.345 62.14) (width 0.25) (layer "F.Cu") (net 3))
-  (segment (start 152.4 51.435) (end 152.4 52.56637) (width 0.25) (layer "F.Cu") (net 3))
+  (segment (start 152.4 56.896) (end 152.4 51.435) (width 0.25) (layer "F.Cu") (net 3))
+  (segment (start 140.97 49.53) (end 144.145 46.355) (width 0.25) (layer "F.Cu") (net 3))
+  (segment (start 137.17 60.965) (end 138.345 62.14) (width 0.25) (layer "F.Cu") (net 3))
   (segment (start 103.135 66.305) (end 100.965 64.135) (width 0.25) (layer "F.Cu") (net 3))
+  (segment (start 138.345 62.14) (end 147.156 62.14) (width 0.25) (layer "F.Cu") (net 3))
+  (segment (start 140.97 61.366701) (end 140.97 49.53) (width 0.25) (layer "F.Cu") (net 3))
   (segment (start 100.965 64.135) (end 102.09 63.01) (width 0.25) (layer "B.Cu") (net 3))
   (segment (start 102.09 63.01) (end 115.08 63.01) (width 0.25) (layer "B.Cu") (net 3))
@@
   (segment (start 122.240991 57.15) (end 121.750991 57.64) (width 0.25) (layer "F.Cu") (net 5))
   (segment (start 139.71 60.965) (end 138.345 59.6) (width 0.25) (layer "F.Cu") (net 5))
-  (segment (start 138.535 59.6) (end 119.29 59.6) (width 0.25) (layer "B.Cu") (net 6))
-  (segment (start 119.29 59.6) (end 116.205 56.515) (width 0.25) (layer "B.Cu") (net 6))
-  (segment (start 139.71 58.425) (end 138.535 59.6) (width 0.25) (layer "B.Cu") (net 6))
+  (segment (start 125.476 55.372) (end 129.704 59.6) (width 0.25) (layer "B.Cu") (net 6))
+  (segment (start 116.205 56.515) (end 117.348 55.372) (width 0.25) (layer "B.Cu") (net 6))
+  (segment (start 138.535 59.6) (end 139.71 58.425) (width 0.25) (layer "B.Cu") (net 6))
+  (segment (start 129.704 59.6) (end 138.535 59.6) (width 0.25) (layer "B.Cu") (net 6))
+  (segment (start 117.348 55.372) (end 125.476 55.372) (width 0.25) (layer "B.Cu") (net 6))
   (segment (start 152.4 34.29) (end 152.4 41.275) (width 0.25) (layer "F.Cu") (net 8))
-  (segment (start 152.4 41.275) (end 152.4 48.275) (width 0.25) (layer "F.Cu") (net 8))
-  (segment (start 152.4 48.275) (end 142.25 58.425) (width 0.25) (layer "F.Cu") (net 8))
+  (segment (start 152.4 48.275) (end 152.4 41.275) (width 0.25) (layer "F.Cu") (net 8))
+  (segment (start 142.25 58.425) (end 152.4 48.275) (width 0.25) (layer "F.Cu") (net 8))
   (segment (start 104.92 63.01) (end 106.045 64.135) (width 0.25) (layer "F.Cu") (net 12))
   (segment (start 83.82 50.801396) (end 96.028604 63.01) (width 0.25) (layer "F.Cu") (net 12))
