File: kiosk/electronics/iowa-rover-kiosk-level-buttons/iowa-rover-kiosk-level-buttons.kicad_pcb (KiCad board)
At the start: 2 copper layers, 137.8 x 41.3 mm, 30 parts, among them J1 Conn_02x08_Top_Bottom, SW1 SW_Push, SW2 SW_Push, SW3 SW_Push, SW4 SW_Push, SW5 SW_Push, SW6 SW_Push, SW7 SW_Push, SW8 SW_Push, U2 TPIC6B595

Commit message: update
Parts:
- Btn Down 1: renamed from SW2
- Btn Down 2: renamed from SW4
- Btn Down 3: renamed from SW6
- Btn Down 4: renamed from SW8
- Btn Up 1: renamed from SW1
- Btn Up 2: renamed from SW3
- Btn Up 3: renamed from SW5
- Btn Up 4: renamed from SW7
- Lamp Down 1: renamed from LA2
- Lamp Down 2: renamed from LA4
- Lamp Down 3: renamed from LA6
- Lamp Down 4: renamed from LA8
- Lamp Up 1: renamed from LA1
- Lamp Up 2: renamed from LA3
- Lamp Up 3: renamed from LA5
- Lamp Up 4: renamed from LA7
Connections:
- Lamp Down 1 pad 2: +12V -> +5V
- Lamp Down 2 pad 2: +12V -> +5V
- Lamp Down 3 pad 2: +12V -> +5V
- Lamp Down 4 pad 2: +12V -> +5V
- Lamp Up 1 pad 2: +12V -> +5V
- Lamp Up 2 pad 2: +12V -> +5V
- Lamp Up 3 pad 2: +12V -> +5V
- Lamp Up 4 pad 2: +12V -> +5V
Routing:
- net +5V: track 202.2 -> 370.9 mm
- net +12V: track 154.2 -> 0.00 mm
Other:
- board text added: "+"
