File: rover/electronics/iowa-rover/iowa-rover.kicad_pcb (KiCad board)
At the start: 2 copper layers, 10 parts, among them J1 Adafruit_USB_C, J2 Conn_01x02, J3 Conn_01x02, U1 Adafruit_Metro_Mini, U2 Adafruit_RFM69HCW_Breakout, U3 Adafruit_TB6612_Breakout

Commit message: draw board
Parts:
- added REF**: MountingHole_2.5mm, MountingHole:MountingHole_2.5mm, F.Cu at (91.0, 153.0)
- added REF**: MountingHole_2.5mm, MountingHole:MountingHole_2.5mm, F.Cu at (43.0, 64.5)
- added REF**: MountingHole_2.5mm, MountingHole:MountingHole_2.5mm, F.Cu at (43.0, 153.0)
- added REF**: MountingHole_2.5mm, MountingHole:MountingHole_2.5mm, F.Cu at (91.0, 64.5)
- moved J2 106.7 mm to (43.2, 99.1), turned to -90 degrees
- moved U3 72.8 mm to (61.0, 96.5), turned to 180 degrees
- moved U1 52.6 mm to (76.2, 106.7)
- moved J3 51.2 mm to (43.2, 111.8), turned to -90 degrees
- moved C1 34.1 mm to (49.0, 71.2), turned to -90 degrees
- moved RV1 33.5 mm to (81.3, 88.4), turned to 90 degrees
- moved U2 13.7 mm to (68.6, 144.8), turned to 90 degrees
- moved R1 0.51 mm to (42.7, 81.3)
Connections:
- net Net-(J2-Pad1) renamed /MA1
- net Net-(J2-Pad2) renamed /MA2
- net Net-(J3-Pad1) renamed /MB1
- net Net-(J3-Pad2) renamed /MB2
- J1 pad S1: unconnected-(J1-PadS1) -> GND
Routing:
- net +5V: track 0.00 -> 105.4 mm
- net /PWMA: track 0.00 -> 53.3 mm
- net Net-(U1-A0): track 0.00 -> 52.8 mm
- net /RADIO_RESET: track 0.00 -> 47.2 mm
- net /AIN1: track 0.00 -> 43.3 mm
- net /AIN2: track 0.00 -> 42.7 mm
- net /RADIO_CLOCK: track 0.00 -> 41.7 mm
- net /RADIO_MISO: track 0.00 -> 36.0 mm
- net /PWMB: track 0.00 -> 33.9 mm
- net /BIN1: track 0.00 -> 33.1 mm
- net /RADIO_MOSI: track 0.00 -> 30.2 mm
- net /BIN2: track 0.00 -> 27.7 mm
- net Net-(U1-3V3): track 0.00 -> 25.5 mm
- net /RADIO_INT: track 0.00 -> 25.0 mm
- net /RADIO_CS: track 0.00 -> 24.8 mm
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- added copper zone on B.Cu, net GND
- added copper zone on In1.Cu, net GND
Other:
- board outline added: 56.3 x 95.9 mm
- copper layers 2 -> 4

Commit message: generate gerbers
Parts:
- added G***: LOGO, SMM:smm-logo-15mm, F.Cu at (74.9, 66.0)
- moved R1 17.7 mm to (57.1, 71.1), turned to 0 degrees
- moved J2 16.6 mm to (44.5, 82.5)
- moved J3 16.6 mm to (44.5, 95.2)
- moved U3 14.4 mm to (71.1, 106.7)
- moved R2 13.1 mm to (57.1, 74.9), turned to 0 degrees
Routing:
- net Net-(J1-CC1): track 10.1 -> 20.5 mm
- net Net-(J1-CC2): track 9.28 -> 17.5 mm
- net /MB2: track 19.4 -> 12.0 mm
- net /MA2: track 17.1 -> 13.0 mm
- net /MB1: track 16.9 -> 13.0 mm
Other:
- board text added: "Rover Controller Rev 0"

Commit message: update
Parts:
- added SW1: SW_SPDT, SMM:SW_EG1218, F.Cu at (65.4, 114.3)
Connections:
- U1 pad 10: unconnected-(U1-A1-Pad10) -> Net-(SW1-B)
Routing:
- net Net-(SW1-B): track 0.00 -> 19.7 mm
Other:
- board text added: "1"
- board text added: "2"
- board text added: "Kiosk Select"
- board text added: "Rover Controller Rev 1a"
- board text removed: "Rover Controller Rev 0"
Changed lines of the file:
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@@
   (net 11 "unconnected-(U1-A3-Pad12)")
   (net 12 "unconnected-(U1-A2-Pad11)")
-  (net 13 "unconnected-(U1-A1-Pad10)")
+  (net 13 "Net-(SW1-B)")
   (net 14 "unconnected-(U1-AREF-Pad8)")
   (net 15 "unconnected-(U1-VIN-Pad7)")
@@
       (net 6 "Net-(U1-A0)") (pinfunction "A0") (pintype "bidirectional"))
     (pad "10" thru_hole circle (at 0 22.86) (size 1.524 1.524) (drill 0.762) (layers "*.Cu" "*.Mask")
-      (net 13 "unconnected-(U1-A1-Pad10)") (pinfunction "A1") (pintype "bidirectional+no_connect"))
+      (net 13 "Net-(SW1-B)") (pinfunction "A1") (pintype "bidirectional"))
     (pad "11" thru_hole circle (at 0 25.4) (size 1.524 1.524) (drill 0.762) (layers "*.Cu" "*.Mask")
       (net 12 "unconnected-(U1-A2-Pad11)") (pinfunction "A2") (pintype "bidirectional+no_connect"))
@@
     (pad "28" thru_hole circle (at 15.24 0) (size 1.524 1.524) (drill 0.762) (layers "*.Cu" "*.Mask")
       (net 30 "/RADIO_CLOCK") (pinfunction "D13") (pintype "bidirectional"))
+  )
+  (footprint "SMM:SW_EG1218" (layer "F.Cu")
+    (at 65.405 114.3 -90)
+    (descr "Through hole straight pin header, 1x03, 2.54mm pitch, single row")
+    (tags "Through hole pin header THT 1x03 2.54mm single row")
+    (property "Sheetfile" "iowa-rover.kicad_sch")
+    (property "Sheetname" "")
+    (property "ki_description" "Switch, single pole double throw")
+    (property "ki_keywords" "switch single-pole double-throw spdt ON-ON")
+    (attr through_hole)
+    (fp_text reference "SW1" (at -3.81 0) (layer "F.SilkS")
+        (effects (font (size 1 1) (thickness 0.15)))
+    )
+    (fp_text value "SW_SPDT" (at 0 7.41 90) (layer "F.Fab")
+        (effects (font (size 1 1) (thickness 0.15)))
+    )
+    (fp_text user "${REFERENCE}" (at -6.35 2.54) (layer "F.Fab")
+        (effects (font (size 1 1) (thickness 0.15)))
+    )
+    (fp_rect (start -2 -5.885) (end 2 6.35)
+      (stroke (width 0.1) (type default)) (fill none) (layer "F.SilkS"))
+    (fp_line (start -1.8 -4.34) (end -1.8 4.31)
+      (stroke (width 0.05) (type solid)) (layer "F.CrtYd"))
+    (fp_line (start -1.8 4.31) (end 1.8 4.31)
+      (stroke (width 0.05) (type solid)) (layer "F.CrtYd"))
+    (fp_line (start 1.8 -4.34) (end -1.8 -4.34)
+      (stroke (width 0.05) (type solid)) (layer "F.CrtYd"))
+    (fp_line (start 1.8 4.31) (end 1.8 -4.34)
+      (stroke (width 0.05) (type solid)) (layer "F.CrtYd"))
+    (fp_rect (start -2 -5.885) (end 2 6.35)
+      (stroke (width 0.1) (type default)) (fill none) (layer "F.Fab"))
+    (pad "1" thru_hole rect (at 0 -2.54 270) (size 1.7 1.7) (drill 1) (layers "*.Cu" "*.Mask")
+      (net 1 "+5V") (pinfunction "A") (pintype "passive"))
+    (pad "2" thru_hole oval (at 0 0 270) (size 1.7 1.7) (drill 1) (layers "*.Cu" "*.Mask")
+      (net 13 "Net-(SW1-B)") (pinfunction "B") (pintype "passive"))
+    (pad "3" thru_hole oval (at 0 2.54 270) (size 1.7 1.7) (drill 1) (layers "*.Cu" "*.Mask")
+      (net 2 "GND") (pinfunction "C") (pintype "passive"))
+    (model "${KICAD6_3DMODEL_DIR}/Connector_PinHeader_2.54mm.3dshapes/PinHeader_1x03_P2.54mm_Vertical.wrl"
+      (offset (xyz 0 0 0))
+      (scale (xyz 1 1 1))
+      (rotate (xyz 0 0 0))
+    )
   )
   (footprint "SMM:smm-logo-15mm" (layer "F.Cu")
@@
     )
   )
+  (gr_poly
+    (pts
+      (xy 57.15 113.665)
+      (xy 58.42 114.3)
+      (xy 57.15 114.935)
+    )
+    (stroke (width 0.15) (type solid)) (fill solid) (layer "F.SilkS"))
   (gr_rect (start 39.116 60.754) (end 95.377 156.67)
     (stroke (width 0.1) (type default)) (fill none) (layer "Edge.Cuts"))
-  (gr_text "Rover Controller Rev 0" (at 48.26 64.77) (layer "F.SilkS")
+  (gr_text "Rover Controller Rev 1a" (at 48.26 64.77) (layer "F.SilkS")
     (effects (font (size 1 1) (thickness 0.15)) (justify left bottom))
   )
+  (gr_text "Kiosk Select" (at 46.99 114.935) (layer "F.SilkS")
+    (effects (font (size 1 1) (thickness 0.25) bold) (justify left bottom))
+  )
+  (gr_text "1" (at 59.69 118.11) (layer "F.SilkS")
+    (effects (font (size 1 1) (thickness 0.25) bold) (justify left bottom))
+  )
+  (gr_text "2" (at 69.85 118.11) (layer "F.SilkS")
+    (effects (font (size 1 1) (thickness 0.25) bold) (justify left bottom))
+  )
   (segment (start 48.022 72.16) (end 49.022 71.16) (width 0.5) (layer "F.Cu") (net 1))
-  (segment (start 62.992 125.984) (end 62.992 140.26963) (width 1.38) (layer "F.Cu") (net 1))
+  (segment (start 62.865 119.38) (end 62.865 140.14263) (width 1.38) (layer "F.Cu") (net 1))
   (segment (start 45.09 75.16) (end 46.09 75.16) (width 0.5) (layer "F.Cu") (net 1))
   (segment (start 45.09 72.16) (end 48.022 72.16) (width 0.5) (layer "F.Cu") (net 1))
   (segment (start 46.09 75.16) (end 49.022 72.228) (width 0.5) (layer "F.Cu") (net 1))
+  (segment (start 71.12 106.68) (end 71.12 111.125) (width 1.38) (layer "F.Cu") (net 1))
   (segment (start 49.022 72.228) (end 49.022 71.16) (width 0.5) (layer "F.Cu") (net 1))
+  (segment (start 71.12 111.125) (end 62.865 119.38) (width 1.38) (layer "F.Cu") (net 1))
   (segment (start 48.935 71.16) (end 48.895 71.12) (width 0.5) (layer "F.Cu") (net 1))
-  (segment (start 71.12 117.856) (end 62.992 125.984) (width 1.38) (layer "F.Cu") (net 1))
-  (segment (start 71.12 106.68) (end 71.12 117.856) (width 1.38) (layer "F.Cu") (net 1))
+  (segment (start 76.2 106.68) (end 71.12 106.68) (width 1.38) (layer "F.Cu") (net 1))
+  (segment (start 71.12 104.14) (end 71.12 106.68) (width 1.38) (layer "F.Cu") (net 1))
+  (segment (start 62.865 140.14263) (end 67.50237 144.78) (width 1.38) (layer "F.Cu") (net 1))
   (segment (start 67.50237 144.78) (end 68.58 144.78) (width 1.38) (layer "F.Cu") (net 1))
-  (segment (start 76.2 106.68) (end 71.12 106.68) (width 1.38) (layer "F.Cu") (net 1))
-  (segment (start 62.992 140.26963) (end 67.50237 144.78) (width 1.38) (layer "F.Cu") (net 1))
-  (segment (start 71.12 104.14) (end 71.12 106.68) (width 1.38) (layer "F.Cu") (net 1))
   (segment (start 68.218 90.356) (end 68.218 102.31563) (width 1.38) (layer "In2.Cu") (net 1))
   (segment (start 49.022 71.16) (end 68.218 90.356) (width 1.38) (layer "In2.Cu") (net 1))
@@
   (segment (start 92.527 97.107) (end 92.527 117.290251) (width 0.25) (layer "F.Cu") (net 6))
   (segment (start 86.177 118.293) (end 77.47 127) (width 0.25) (layer "F.Cu") (net 6))
+  (segment (start 65.405 118.745) (end 76.2 129.54) (width 0.25) (layer "In2.Cu") (net 13))
+  (segment (start 65.405 114.3) (end 65.405 118.745) (width 0.25) (layer "In2.Cu") (net 13))
   (segment (start 68.129749 143.327) (end 82.733 143.327) (width 0.25) (layer "F.Cu") (net 19))
   (segment (start 66.593 126.447) (end 66.593 141.790251) (width 0.25) (layer "F.Cu") (net 19))
