File: kiosk/electronics/iowa-rover-kiosk-main/iowa-rover-kiosk-main.kicad_sch (KiCad schematic)
At the start: 13 parts, among them J1 Conn_01x04, J1 Conn_01x08, J1 Conn_02x08_Top_Bottom, J2 Barrel_Jack, J3 Conn_02x06_Odd_Even, J7 Conn_01x03, U1 Adafruit_RFM69HCW_Breakout, U2 I50115, U3 ATtiny84-20P

Commit message: update
Connections:
- net SCL: now also U3.9 (PA4); no longer U3.7 (PA6)
- net SDA: now also U3.7 (PA6); no longer U3.9 (PA4)
Changed lines of the file:
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@@
     (effects (font (size 1.27 1.27)) (justify left bottom))
   )
-  (label "SCL" (at 204.47 83.82 0) (fields_autoplaced)
+  (label "SCL" (at 204.47 78.74 0) (fields_autoplaced)
     (effects (font (size 1.27 1.27)) (justify left bottom))
   )
@@
     (effects (font (size 1.27 1.27)) (justify left bottom))
   )
-  (label "SDA" (at 204.47 78.74 0) (fields_autoplaced)
+  (label "SDA" (at 204.47 83.82 0) (fields_autoplaced)
     (effects (font (size 1.27 1.27)) (justify left bottom))
   )

Commit message: add pdf schematics
Other:
- company: (none) -> Science Museum of Minnesota
- title: (none) -> Iowa Science Rover Kiosk - Main Board
Changed lines of the file:
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@@
 (kicad_sch (version 20230121) (generator eeschema)
   (paper "A4")
+  (title_block
+    (title "Iowa Science Rover Kiosk - Main Board")
+    (date "2023-10-05")
+    (rev "0")
+    (company "Science Museum of Minnesota")
+    (comment 1 "Kate Swanson")
+  )
   (junction (at 60.96 48.895) (diameter 0) (color 0 0 0 0)
   )
