File: kiosk/electronics/iowa-rover-kiosk-mega-adapter/iowa-rover-kiosk-mega-adapter.kicad_sch (KiCad schematic)
At the start: 2 parts

Commit message: add pdf schematics
Other:
- company: (none) -> Science Museum of Minnesota
- title: (none) -> Iowa Science Rover Kiosk - Mega Adapter Board
Changed lines of the file:
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@@
 (kicad_sch (version 20230121) (generator eeschema)
   (paper "A4")
+  (title_block
+    (title "Iowa Science Rover Kiosk - Mega Adapter Board")
+    (date "2023-10-05")
+    (rev "0")
+    (company "Science Museum of Minnesota")
+    (comment 1 "Kate Swanson")
+  )
   (junction (at 38.1 149.225) (diameter 0) (color 0 0 0 0)
   )
