File: kiosk/electronics/iowa-rover-kiosk-programmer/iowa-rover-kiosk-programmer.kicad_sch (KiCad schematic)
At the start: 20 parts

Commit message: update
Parts:
- D1, D2, D3, D4: value (none) -> LED; footprint (none) -> LED_THT:LED_D3.0mm
- J1: value (none) -> Conn_02x06_Odd_Even; footprint (none) -> Connector_PinHeader_2.54mm:PinHeader_2x06_P2.54mm_Vertical
- R1, R2, R3, R4: value (none) -> 1k; footprint (none) -> Resistor_THT:R_Axial_DIN0207_L6.3mm_D2.5mm_P10.16mm_Horizontal
- R5, R6, R7, R8, R9: value (none) -> 10k; footprint (none) -> Resistor_THT:R_Axial_DIN0207_L6.3mm_D2.5mm_P10.16mm_Horizontal
- SW1, SW2, SW3, SW4, SW5: value (none) -> SW_Push; footprint (none) -> Button_Switch_THT:SW_PUSH_6mm_H4.3mm
- U1: value (none) -> ID12-LA; footprint (none) -> SMM:ID-12LA

Commit message: add pdf schematics
Other:
- company: (none) -> Science Museum of Minnesota
- title: (none) -> Iowa Science Rover Kiosk - RFID Programmer Board
Changed lines of the file:
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@@
 (kicad_sch (version 20230121) (generator eeschema)
   (paper "A4")
+  (title_block
+    (title "Iowa Science Rover Kiosk - RFID Programmer Board")
+    (date "2023-10-05")
+    (rev "0")
+    (company "Science Museum of Minnesota")
+    (comment 1 "Kate Swanson")
+  )
   (junction (at 102.87 109.22) (diameter 0) (color 0 0 0 0)
   )
