File: kiosk/electronics/iowa-rover-kiosk-power-cycler/iowa-rover-kiosk-power-cycler.kicad_sch (KiCad schematic)
At the start: 5 parts, among them J1 Conn_01x04, J2 Conn_01x04, Q1 IRF40B207, U1 ATtiny85-20P

Commit message: add power cycler kiosk pdf
Other:
- company: (none) -> Science Museum of Minnesota
- title: (none) -> Iowa Rover Kiosk - Power Cycler Board
Changed lines of the file:
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@@
 (kicad_sch (version 20230121) (generator eeschema)
   (paper "A4")
+  (title_block
+    (title "Iowa Rover Kiosk - Power Cycler Board")
+    (date "2023-12-21")
+    (rev "0")
+    (company "Science Museum of Minnesota")
+    (comment 1 "Kate Swanson")
+  )
   (junction (at 134.62 54.61) (diameter 0) (color 0 0 0 0)
   )
